File: projekt/projekt.kicad_pcb (KiCad board)
At the start: 2 copper layers, 19 parts, among them J1 S8421-45R, SW1 SW_Push, U1 NE555P

Commit message: wow! serduszko!
Parts:
- added C2: 10n, Capacitor_THT:C_Disc_D4.3mm_W1.9mm_P5.00mm, F.Cu at (181.0, 84.0)
- added R3: 100, Resistor_THT:R_Axial_DIN0207_L6.3mm_D2.5mm_P7.62mm_Horizontal, F.Cu at (174.8, 60.0)
- added R4: 100, Resistor_THT:R_Axial_DIN0207_L6.3mm_D2.5mm_P7.62mm_Horizontal, F.Cu at (175.3, 66.5)
- moved D7 64.4 mm to (170.0, 125.4), turned to -90 degrees
- moved D9 64.3 mm to (150.0, 106.4), turned to 90 degrees
- moved D6 57.4 mm to (183.9, 115.5)
- moved D8 55.4 mm to (157.6, 116.0)
- moved D10 54.2 mm to (143.6, 90.0)
- moved D11 47.4 mm to (141.8, 75.0)
- moved D5 44.4 mm to (196.4, 96.0)
- moved D12 36.9 mm to (151.1, 60.0)
- moved R2 29.5 mm to (188.9, 79.3)
- moved D4 28.3 mm to (201.4, 77.1)
- moved R1 25.0 mm to (174.9, 72.5)
- moved D3 24.1 mm to (198.9, 67.5)
- moved SW1 22.8 mm to (172.2, 113.0)
- moved J1 22.5 mm to (169.0, 100.0)
- moved U1 21.6 mm to (174.0, 77.2)
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Connections:
- D1 pad 1: GND -> Net-(D1-K)
- D1 pad 2: Net-(D1-A) -> /OUT
- D10 pad 2: VCC -> Net-(D10-A)
- D11 pad 1: GND -> Net-(D1-K)
- D11 pad 2: Net-(D1-A) -> /OUT
- D12 pad 1: Net-(D1-A) -> /OUT
- D12 pad 2: VCC -> Net-(D10-A)
- D2 pad 1: Net-(D1-A) -> /OUT
- D2 pad 2: VCC -> Net-(D10-A)
- D3 pad 1: GND -> Net-(D1-K)
- D4 pad 2: VCC -> Net-(D10-A)
- D5 pad 1: GND -> Net-(D1-K)
- D6 pad 2: VCC -> Net-(D10-A)
- D7 pad 1: GND -> Net-(D1-K)
- D8 pad 2: VCC -> Net-(D10-A)
- D9 pad 1: GND -> Net-(D1-K)
- U1 pad 5: GND -> Net-(U1-CV)
Other:
- board outline added: 70 x 73.4 mm

Commit message: serduszko nawet bardziej
Parts:
- moved R3 27.4 mm to (153.4, 77.0)
- moved D9 9.16 mm to (144.0, 99.5), turned to -60 degrees
- moved D11 8.05 mm to (141.0, 67.0), turned to 55 degrees
- moved D10 7.86 mm to (138.5, 84.0), turned to -77.5 degrees
- moved SW1 7.81 mm to (173.2, 120.8), turned to 180 degrees
- moved D4 6.93 mm to (201.5, 84.0), turned to 77.5 degrees
- moved R3 4.97 mm to (187.2, 88.0)
- moved D12 4.45 mm to (155.5, 59.5), turned to -2.5 degrees
- moved D2 4.11 mm to (184.5, 59.5), turned to 2.5 degrees
- moved D5 3.53 mm to (196.0, 99.5), turned to 60 degrees
- moved D8 3.23 mm to (154.5, 115.0), turned to -48 degrees
- moved J1 2.24 mm to (168.0, 102.0)
- moved D6 1.65 mm to (185.5, 115.0), turned to 48 degrees
- moved D7 1.08 mm to (170.0, 126.5), turned to 0 degrees
- moved D3 0.51 mm to (199.0, 67.0), turned to -55 degrees

Commit message: wiekszy margines od kranca swiata
Parts:
- removed the R3 at (187.2, 88.0)
- moved D10 0.50 mm to (139.0, 84.0)
- moved D11 0.50 mm to (141.5, 67.0)
- moved D3 0.50 mm to (198.5, 67.0)
- moved D4 0.50 mm to (201.0, 84.0)
- moved D5 0.50 mm to (195.5, 99.5), turned to -120 degrees
- moved D6 0.50 mm to (185.0, 115.0)
- moved D7 0.50 mm to (170.0, 126.0), turned to 180 degrees
- moved D8 0.50 mm to (155.0, 115.0)
- moved D9 0.50 mm to (144.5, 99.5), turned to 120 degrees
- moved D12 0.44 mm to (155.5, 59.9), turned to 177.5 degrees
- moved D2 0.44 mm to (184.5, 59.9), turned to -177.5 degrees
Connections:
- net Net-(D1-K) renamed /L_GND
- net Net-(D10-A) renamed /L_VCC
- D10 pad 1: Net-(D10-K) -> /OUT
- D3 pad 2: Net-(D3-A) -> /OUT
- D4 pad 1: Net-(D3-A) -> /OUT
- D5 pad 2: Net-(D5-A) -> /OUT
- D6 pad 1: Net-(D5-A) -> /OUT
- D7 pad 2: Net-(D7-A) -> /OUT
- D8 pad 1: Net-(D7-A) -> /OUT
- D9 pad 2: Net-(D10-K) -> /OUT

Commit message: pierscien
Parts:
- moved SW1 97.5 mm to (270.0, 108.5)
- moved J1 92.7 mm to (256.5, 129.5)
- moved C1 85.3 mm to (236.0, 102.0)
- moved R3 85.3 mm to (231.4, 111.5)
- moved U1 74.2 mm to (245.6, 57.7)
- moved C2 73.7 mm to (251.3, 62.0)
- moved R1 68.8 mm to (242.5, 85.3)
- moved R2 68.8 mm to (256.5, 92.1)
- moved R4 68.8 mm to (242.9, 79.3)
- moved D1 0.15 mm to (170.0, 66.5)
Routing:
- net /OUT: track 0.00 -> 251.2 mm

Commit message: ja pd udało sie - wszystkie połączenia zrobione
Parts:
- moved SW1 103.3 mm to (166.8, 107.8), turned to 0 degrees
- moved J1 93.1 mm to (170.0, 95.0)
- moved R4 88.1 mm to (157.0, 98.8), turned to 90 degrees
- moved C2 81.6 mm to (172.5, 83.0), turned to 180 degrees
- moved U1 80.7 mm to (166.2, 72.2), turned to 0 degrees
- moved C1 79.9 mm to (161.8, 72.2)
- moved R2 79.2 mm to (180.0, 71.7), turned to -90 degrees
- moved R1 66.9 mm to (177.0, 71.7), turned to -90 degrees
- moved R3 46.9 mm to (186.2, 98.8), turned to 90 degrees
- moved D12 0.31 mm to (155.5, 60.2)
- moved D2 0.31 mm to (184.5, 60.2)
- turned D1 to -90 degrees
Routing:
- net /L_GND: track 0.00 -> 254.3 mm, vias 0 -> 1
- net /L_VCC: track 0.00 -> 224.6 mm
- net VCC: track 0.00 -> 74.4 mm
- net GND: track 0.00 -> 49.2 mm
- net Net-(U1-THR): track 0.00 -> 23.7 mm
- net /OUT: track 251.2 -> 271.5 mm
- net Net-(J1-PadP): track 0.00 -> 16.7 mm
- net Net-(U1-DIS): track 0.00 -> 12.9 mm
- net Net-(U1-CV): track 0.00 -> 3.73 mm
