File: projekt/projekt.kicad_pcb (KiCad board)
At the start: 2 copper layers, 70 x 73.4 mm, 21 parts, among them J1 S8421-45R, SW1 SW_Push, U1 NE555P

Commit message: wieksze dziury
Other:
- board text added: "Wesołych"
- board text added: "Świąt!"
Changed lines of the file:
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@@
 		(pad "1" thru_hole roundrect
 			(at 0 0)
-			(size 1.2 1.2)
+			(size 1.6 1.6)
 			(drill 0.6)
 			(layers "*.Cu" "*.Mask")
@@
 		(pad "2" thru_hole circle
 			(at 2 0)
-			(size 1.2 1.2)
+			(size 1.6 1.6)
 			(drill 0.6)
 			(layers "*.Cu" "*.Mask")
@@
 		(attr smd)
 		(fp_line
-			(start -2.5 -1.399999)
+			(start -2.5 -1.399998)
 			(end -2.5 1.4)
 			(stroke
@@
 		(fp_line
 			(start 2.2 -1.4)
-			(end -2.5 -1.399999)
+			(end -2.5 -1.399998)
 			(stroke
 				(width 0.12)
@@
 		(fp_line
 			(start -0.55 -0.7)
-			(end 0.550001 -0.7)
+			(end 0.550002 -0.7)
 			(stroke
 				(width 0.1)
@@
 		)
 		(fp_line
-			(start -0.550001 0.7)
+			(start -0.550002 0.7)
 			(end 0.55 0.7)
 			(stroke
@@
 		)
 		(fp_arc
-			(start 0.550001 -0.7)
+			(start 0.550002 -0.7)
 			(mid 1.25 0)
 			(end 0.55 0.7)
@@
 		)
 		(fp_arc
-			(start -0.550001 0.7)
+			(start -0.550002 0.7)
 			(mid -1.25 0)
 			(end -0.55 -0.7)
@@
 		(layer "User.1")
 	)
+	(gr_text "Wesołych"
+		(at 152.5 90 90)
+		(layer "F.Cu")
+		(effects
+			(font
+				(size 3 3)
+				(thickness 0.6)
+				(bold yes)
+			)
+			(justify left bottom)
+		)
+	)
+	(gr_text "Świąt!"
+		(at 187.5 72.5 270)
+		(layer "F.Cu")
+		(effects
+			(font
+				(size 3 3)
+				(thickness 0.6)
+				(bold yes)
+			)
+			(justify left bottom)
+		)
+	)
 	(segment

Commit message: V3! grubsze wszystko!
Parts:
- moved D7 2.25 mm to (170.0, 123.8)
- moved D10 2.24 mm to (141.0, 85.0)
- moved D11 2.24 mm to (142.5, 69.0)
- moved D3 2.24 mm to (197.5, 69.0)
- moved D4 2.24 mm to (199.0, 85.0)
- moved D6 1.80 mm to (184.0, 113.5)
- moved D8 1.80 mm to (156.0, 113.5)
- moved D5 1.75 mm to (193.8, 99.5)
- moved D9 1.75 mm to (146.2, 99.5)
- moved D1 1.50 mm to (170.0, 68.0)
- moved D12 1.50 mm to (155.5, 61.8)
- moved D2 1.50 mm to (184.5, 61.8)
Routing:
- net /L_VCC: track 224.6 -> 189.4 mm, vias 0 -> 2
- net /OUT: track 271.5 -> 285.5 mm
- net /L_GND: track 254.3 -> 260.6 mm
- net Net-(U1-THR): track 23.7 -> 21.8 mm
- net GND: track 49.2 -> 47.5 mm
- net VCC: track 74.4 -> 75.4 mm

Commit message: forgor
Routing:
- net /L_VCC: track 189.4 -> 200.4 mm
Changed lines of the file:
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@@
+	)
+	(segment
+		(start 175.5 65)
+		(end 164.5 65)
+		(width 0.8)
+		(layer "B.Cu")
+		(net 5)
 	)
 	(segment
