File: projekt/projekt.kicad_sch (KiCad schematic)
At the start: 20 parts, among them J1 S8421-45R, SW1 SW_Push, U1 NE555P

Commit message: make it kinda work
Parts:
- added C2: 10n, symbol Device:C
- added R4: 100, Resistor_THT:R_Axial_DIN0207_L6.3mm_D2.5mm_P7.62mm_Horizontal, symbol Device:R
- R3: value R -> 100
Connections:
- net GND: now also R3.2, C2.2; no longer D1.1 (K), D11.1 (K), D3.1 (K), D5.1 (K), D7.1 (K), D9.1 (K), U1.5 (CV)
- net OUT: now also D1.2 (A), D11.2 (A), D12.1 (K), D2.1 (K); no longer R3.1
- net VCC: now also R4.1; no longer D10.2 (A), D12.2 (A), D2.2 (A), D4.2 (A), D6.2 (A), D8.2 (A)
- new net: D10.2 (A), D12.2 (A), D2.2 (A), D4.2 (A), D6.2 (A), D8.2 (A), R4.2
- new net: D1.1 (K), D11.1 (K), D3.1 (K), D5.1 (K), D7.1 (K), D9.1 (K), R3.1
- new net: C2.1, U1.5 (CV)
Other:
- moved on the sheet: D1, D10, D11, D12, D2, D3, D4, D5, D6, D7, D8, D9

Commit message: wow! serduszko!
Parts:
- C2: footprint (none) -> Capacitor_THT:C_Disc_D4.3mm_W1.9mm_P5.00mm
- renumbered R4 to R3, R3 to R4
Changed lines of the file:
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@@
 		(dnp no)
 		(fields_autoplaced yes)
-		(property "Reference" "R3"
+		(property "Reference" "R4"
 			(at 166.37 119.3799 0)
 			(effects
@@
 			(project "projekt"
 				(path "/b670f8c9-b4be-4d7f-9216-860ddbeab6b3"
-					(reference "R3")
+					(reference "R4")
 					(unit 1)
 				)
@@
 			)
 		)
-		(property "Footprint" ""
+		(property "Footprint" "Capacitor_THT:C_Disc_D4.3mm_W1.9mm_P5.00mm"
 			(at 113.03 103.1748 0)
 			(effects
@@
 		(dnp no)
 		(fields_autoplaced yes)
-		(property "Reference" "R4"
+		(property "Reference" "R3"
 			(at 191.77 73.6599 0)
 			(effects
@@
 			(project "projekt"
 				(path "/b670f8c9-b4be-4d7f-9216-860ddbeab6b3"
-					(reference "R4")
-					(unit 1)
-				)
+					(reference "R3")
+					(unit 1)
+				)

Commit message: wiekszy margines od kranca swiata
Connections:
- net OUT: now also D10.1 (K), D3.2 (A), D4.1 (K), D5.2 (A), D6.1 (K), D7.2 (A), D8.1 (K), D9.2 (A)
- net L_VCC: now reaches D10.2 (A), D12.2 (A), D2.2 (A), D4.2 (A), D6.2 (A), D8.2 (A), R3.2
- net L_GND: now reaches D1.1 (K), D11.1 (K), D3.1 (K), D5.1 (K), D7.1 (K), D9.1 (K), R4.1
Changed lines of the file:
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@@
+	)
+	(junction
+		(at 176.53 100.33)
+		(diameter 0)
+		(color 0 0 0 0)
+	)
+	(junction
+		(at 163.83 81.28)
+		(diameter 0)
+		(color 0 0 0 0)
 	)
 	(junction
@@
 	)
 	(junction
+		(at 176.53 93.98)
+		(diameter 0)
+		(color 0 0 0 0)
+	)
+	(junction
 		(at 130.81 109.22)
 		(diameter 0)
@@
 	)
 	(junction
+		(at 176.53 87.63)
+		(diameter 0)
+		(color 0 0 0 0)
+	)
+	(junction
 		(at 143.51 92.71)
 		(diameter 0)
@@
 		(color 0 0 0 0)
 	)
+	(junction
+		(at 176.53 106.68)
+		(diameter 0)
+		(color 0 0 0 0)
+	)
 	(wire
 		(pts
@@
 	(wire
 		(pts
-			(xy 176.53 81.28) (xy 176.53 113.03)
+			(xy 176.53 100.33) (xy 179.07 100.33)
+		)
+		(stroke
+			(width 0)
+			(type default)
+		)
+	)
+	(wire
+		(pts
+			(xy 176.53 81.28) (xy 176.53 87.63)
+		)
+		(stroke
+			(width 0)
+			(type default)
+		)
+	)
+	(wire
+		(pts
+			(xy 189.23 81.28) (xy 191.77 81.28)
 		)
 		(stroke
@@
 	(wire
 		(pts
-			(xy 173.99 106.68) (xy 179.07 106.68)
+			(xy 173.99 106.68) (xy 176.53 106.68)
 		)
 		(stroke
@@
 	(wire
 		(pts
+			(xy 176.53 93.98) (xy 179.07 93.98)
+		)
+		(stroke
+			(width 0)
+			(type default)
+		)
+	)
+	(wire
+		(pts
 			(xy 189.23 106.68) (xy 189.23 100.33)
 		)
@@
 	(wire
 		(pts
+			(xy 176.53 87.63) (xy 179.07 87.63)
+		)
+		(stroke
+			(width 0)
+			(type default)
+		)
+	)
+	(wire
+		(pts
 			(xy 99.06 87.63) (xy 99.06 109.22)
 		)
@@
 	(wire
 		(pts
+			(xy 176.53 100.33) (xy 176.53 106.68)
+		)
+		(stroke
+			(width 0)
+			(type default)
+		)
+	)
+	(wire
+		(pts
 			(xy 163.83 116.84) (xy 163.83 113.03)
 		)
@@
 	(wire
 		(pts
-			(xy 173.99 93.98) (xy 179.07 93.98)
+			(xy 173.99 93.98) (xy 176.53 93.98)
 		)
 		(stroke
@@
 	(wire
 		(pts
+			(xy 176.53 93.98) (xy 176.53 100.33)
+		)
+		(stroke
+			(width 0)
+			(type default)
+		)
+	)
+	(wire
+		(pts
 			(xy 163.83 100.33) (xy 163.83 93.98)
 		)
@@
 	(wire
 		(pts
+			(xy 176.53 87.63) (xy 176.53 93.98)
+		)
+		(stroke
+			(width 0)
+			(type default)
+		)
+	)
+	(wire
+		(pts
+			(xy 176.53 106.68) (xy 179.07 106.68)
+		)
+		(stroke
+			(width 0)
+			(type default)
+		)
+	)
+	(wire
+		(pts
 			(xy 163.83 106.68) (xy 166.37 106.68)
 		)
@@
 	(wire
 		(pts
-			(xy 173.99 87.63) (xy 179.07 87.63)
+			(xy 173.99 87.63) (xy 176.53 87.63)
 		)
 		(stroke
@@
 	(wire
 		(pts
+			(xy 176.53 106.68) (xy 176.53 113.03)
+		)
+		(stroke
+			(width 0)
+			(type default)
+		)
+	)
+	(wire
+		(pts
 			(xy 186.69 113.03) (xy 189.23 113.03)
 		)
@@
 	(wire
 		(pts
+			(xy 161.29 81.28) (xy 163.83 81.28)
+		)
+		(stroke
+			(width 0)
+			(type default)
+		)
+	)
+	(wire
+		(pts
 			(xy 163.83 113.03) (xy 163.83 106.68)
 		)
@@
 	(wire
 		(pts
-			(xy 173.99 100.33) (xy 179.07 100.33)
+			(xy 173.99 100.33) (xy 176.53 100.33)
 		)
 		(stroke
@@
 		)
 	)
+	(label "L_GND"
+		(at 161.29 81.28 0)
+		(effects
+			(font
+				(size 1.27 1.27)
+			)
+			(justify left bottom)
+		)
+	)
+	(label "L_VCC"
+		(at 191.77 81.28 0)
+		(effects
+			(font
+				(size 1.27 1.27)
+			)
+			(justify left bottom)
+		)
+	)

Commit message: costam
Parts:
- V1: value 5 -> 10
Changed lines of the file:
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@@
 			)
 		)
-		(property "Value" "5"
+		(property "Value" "10"
 			(at 93.98 133.2201 0)
 			(effects

Commit message: zdjęcia i wgl
Parts:
- V1: value 10 -> 6
Connections:
- net Vcap: now reaches C1.1, R2.2, U1.2 (TR), U1.6 (THR)
Other:
- moved on the sheet: C1, C2, D1, D10, D11, D12, D2, D3, D4, D5, D6, D7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
